File: board/Clock_with_LED.sch (EAGLE design)
At the start: 18 parts

Commit message: Removed LEDs, organised PCB files
Parts:
- added D1, D2: WS2812B, WS2812B:WS2812B
Connections:
- new net N$1: D1.DOUT, D2.DIN
- new net N$2: D1.DIN, SV1.1
- net +5V: now also D1.VDD, D2.VDD, SV1.3; no longer SV1.2
- net GND: now also D1.VSS, D2.VSS, SV1.2; no longer SV1.1
- net N$7: now also D2.DOUT; no longer SV1.3
- net PRG_EN: now also S1.2; no longer S1.1
Other:
- moved on the sheet: SV1
