File: board/Clock_fab.brd (EAGLE design)
At the start: 50 x 50 mm, 20 parts

Commit message: Prepared the PCB for fabrication
Parts:
- removed D1, D2: WS2812B, WS2812B:LED_WS2812B
- C1: value 100uF -> 1000uF; device rcl:TT5D7L -> rcl:TT5D11L
- moved SV1 39.6 mm to (44.1, 10.4)
- moved JP2 12.1 mm to (33.0, 3.56)
- moved PH1 9.96 mm to (13.0, 46.3), turned to 0 degrees
- moved JP1 9.77 mm to (30.5, 3.56)
- moved S1 6.00 mm to (25.0, 5.99), turned to 270 degrees
- moved SV2 4.68 mm to (13.2, 11.2)
- moved C5 4.60 mm to (25.9, 13.7)
- moved C3 3.56 mm to (40.1, 33.0)
- moved C1 2.54 mm to (41.8, 13.2)
- renumbered AMS1117 to REG
Connections:
- removed net GPIO16: R1.1, U$1.12, U$2.S
- removed net N$1: D1.2, D2.4
- removed net N$2: D1.4, SV1.1
- new net GPIO14: R1.1, U$1.13, U$2.S
- net +5V: now also SV1.2; no longer D1.1, D2.1, SV1.3
- net GND: now also SV1.1; no longer D1.3, D2.3, SV1.2
- net N$7: now also SV1.3; no longer D2.2
- net PRG_EN: now also S1.1; no longer S1.2
- net VCC: no longer REG.2
Routing:
- net N$1: track 77.8 -> 8.00 mm, vias 0 -> 1
- net +5V: track 113.3 -> 55.8 mm
- net GND: track 119.3 -> 78.4 mm, vias 0 -> 2
- net N$7: track 35.9 -> 64.7 mm
- net N$5: track 0.00 -> 8.00 mm, vias 0 -> 1
- net N$4: track 0.00 -> 8.00 mm, vias 0 -> 1
- net N$2: track 15.0 -> 8.00 mm, vias 0 -> 1
- net GPIO16: track 5.59 -> 0.00 mm
- net GPIO14: track 0.00 -> 5.11 mm
- net TXD: track 3.26 -> 6.84 mm
- net RXD: track 3.49 -> 6.61 mm
- net PRG_EN: track 15.8 -> 18.1 mm
- net ADC: track 19.0 -> 16.9 mm
- net VCC: track 88.0 -> 90.1 mm
- net REST: track 41.1 -> 42.2 mm
- removed copper zone on layer 16, net N$3
Other:
- outline, holes or cut-outs redrawn
- board text added: "+5V GND"
- board text added: "GND VCC PRG RxD TxD RST"
- board text added: "SYG +5V GND"
- board text removed: "-"
- board text removed: "5V"
