File: board/Clock_fab.sch (EAGLE design)
At the start: 20 parts

Commit message: Prepared the PCB for fabrication
Parts:
- removed D1, D2: WS2812B, WS2812B:WS2812B
- C1: value 100uF -> 1000uF; device rcl:CPOL-EUTT5D7L -> rcl:CPOL-EUTT5D11L
- renumbered AMS1117 to REG
Connections:
- removed net GPIO16: R1.1, U$1.GPIO16, U$2.S
- removed net N$1: D1.DOUT, D2.DIN
- removed net N$2: D1.DIN, SV1.1
- new net GPIO14: R1.1, U$1.GPIO14, U$2.S
- net +5V: now also SV1.2; no longer D1.VDD, D2.VDD, SV1.3
- net GND: now also SV1.1; no longer D1.VSS, D2.VSS, SV1.2
- net N$7: now also SV1.3; no longer D2.DOUT
- net PRG_EN: now also S1.1; no longer S1.2
- net VCC: no longer REG.OUT
Other:
- moved on the sheet: SV1
Changed lines of the file:
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@@
 <parts>
 <part name="U$1" library="ESP8266-ESP12" deviceset="ESP8266_ESP-12" device=""/>
-<part name="AMS1117" library="lm1117" deviceset="LM1117IMPX-*" device="" technology="3.3"/>
+<part name="REG" library="lm1117" deviceset="LM1117IMPX-*" device="" technology="3.3"/>
 <part name="R1" library="rcl" library_urn="urn:adsk.eagle:library:334" deviceset="R-EU_" device="R0805" value="10k"/>
 <part name="R2" library="rcl" library_urn="urn:adsk.eagle:library:334" deviceset="R-EU_" device="R0805" value="10k"/>
@@
 <part name="GND4" library="supply1" library_urn="urn:adsk.eagle:library:371" deviceset="GND" device=""/>
 <part name="GND5" library="supply1" library_urn="urn:adsk.eagle:library:371" deviceset="GND" device=""/>
-<part name="C1" library="rcl" library_urn="urn:adsk.eagle:library:334" deviceset="CPOL-EU" device="TT5D7L" value="100uF"/>
+<part name="C1" library="rcl" library_urn="urn:adsk.eagle:library:334" deviceset="CPOL-EU" device="TT5D11L" value="1000uF"/>
 <part name="C2" library="rcl" library_urn="urn:adsk.eagle:library:334" deviceset="CPOL-EU" device="TT5D7L" value="100uF"/>
 <part name="GND6" library="supply1" library_urn="urn:adsk.eagle:library:371" deviceset="GND" device=""/>
@@
 <part name="P+10" library="supply1" library_urn="urn:adsk.eagle:library:371" deviceset="VCC" device=""/>
 <part name="P+2" library="supply1" library_urn="urn:adsk.eagle:library:371" deviceset="+5V" device=""/>
-<part name="D1" library="WS2812B" deviceset="WS2812B" device=""/>
-<part name="D2" library="WS2812B" deviceset="WS2812B" device=""/>
-<part name="GND7" library="supply1" library_urn="urn:adsk.eagle:library:371" deviceset="GND" device=""/>
-<part name="GND8" library="supply1" library_urn="urn:adsk.eagle:library:371" deviceset="GND" device=""/>
-<part name="P+11" library="supply1" library_urn="urn:adsk.eagle:library:371" deviceset="+5V" device=""/>
-<part name="P+12" library="supply1" library_urn="urn:adsk.eagle:library:371" deviceset="+5V" device=""/>
 <part name="C5" library="rcl" library_urn="urn:adsk.eagle:library:334" deviceset="C-EU" device="C0805" value="10nF"/>
 <part name="P+13" library="supply1" library_urn="urn:adsk.eagle:library:371" deviceset="VCC" device=""/>
@@
 <instances>
 <instance part="U$1" gate="G$1" x="22.86" y="43.18"/>
-<instance part="AMS1117" gate="G$1" x="33.02" y="91.44" smashed="yes">
+<instance part="REG" gate="G$1" x="33.02" y="91.44" smashed="yes">
 <attribute name="NAME" x="25.4" y="99.06" size="1.778" layer="95"/>
 <attribute name="VALUE" x="25.4" y="96.52" size="1.778" layer="96"/>
@@
 <instance part="R3" gate="G$1" x="-2.54" y="58.42" rot="R90"/>
 <instance part="P+3" gate="VCC" x="-2.54" y="68.58"/>
-<instance part="SV1" gate="G$1" x="182.88" y="43.18" rot="MR0"/>
-<instance part="GND4" gate="1" x="172.72" y="35.56" rot="MR0"/>
+<instance part="SV1" gate="G$1" x="109.22" y="38.1" rot="MR0"/>
+<instance part="GND4" gate="1" x="99.06" y="30.48" rot="MR0"/>
 <instance part="GND5" gate="1" x="-2.54" y="78.74"/>
 <instance part="C1" gate="G$1" x="22.86" y="86.36"/>
@@
 <instance part="P+9" gate="1" x="15.24" y="96.52"/>
 <instance part="P+10" gate="VCC" x="50.8" y="96.52"/>
-<instance part="P+2" gate="1" x="172.72" y="50.8" rot="MR0"/>
-<instance part="D1" gate="G$1" x="149.86" y="40.64" rot="MR0"/>
-<instance part="D2" gate="G$1" x="116.84" y="40.64" rot="MR0"/>
-<instance part="GND7" gate="1" x="132.08" y="27.94" rot="MR0"/>
-<instance part="GND8" gate="1" x="99.06" y="27.94" rot="MR0"/>
-<instance part="P+11" gate="1" x="99.06" y="53.34" rot="MR0"/>
-<instance part="P+12" gate="1" x="132.08" y="53.34" rot="MR0"/>
+<instance part="P+2" gate="1" x="99.06" y="45.72" rot="MR0"/>
 <instance part="C5" gate="G$1" x="66.04" y="83.82"/>
 <instance part="P+13" gate="VCC" x="66.04" y="91.44" smashed="yes" rot="MR0">
@@
 <label x="40.64" y="40.64" size="1.27" layer="95" xref="yes"/>
 <wire x1="38.1" y1="40.64" x2="40.64" y2="40.64" width="0.1524" layer="91"/>
-<wire x1="38.1" y1="40.64" x2="38.1" y2="27.94" width="0.1524" layer="91"/>
+<wire x1="38.1" y1="40.64" x2="38.1" y2="30.48" width="0.1524" layer="91"/>
 <junction x="38.1" y="40.64"/>
-<pinref part="S1" gate="G$1" pin="2"/>
-<wire x1="38.1" y1="27.94" x2="43.18" y2="27.94" width="0.1524" layer="91"/>
+<pinref part="S1" gate="G$1" pin="1"/>
+<wire x1="38.1" y1="30.48" x2="43.18" y2="30.48" width="0.1524" layer="91"/>
 </segment>
 <segment>
@@
 <net name="GND" class="0">
 <segment>
-<pinref part="AMS1117" gate="G$1" pin="GND"/>
+<pinref part="REG" gate="G$1" pin="GND"/>
 <pinref part="GND2" gate="1" pin="GND"/>
 <wire x1="33.02" y1="83.82" x2="33.02" y2="78.74" width="0.1524" layer="91"/>
@@
 </segment>
 <segment>
-<pinref part="GND4" gate="1" pin="GND"/>
-<wire x1="172.72" y1="43.18" x2="172.72" y2="38.1" width="0.1524" layer="91"/>
-<pinref part="SV1" gate="G$1" pin="2"/>
-<wire x1="175.26" y1="43.18" x2="172.72" y2="43.18" width="0.1524" layer="91"/>
-</segment>
-<segment>
 <pinref part="GND5" gate="1" pin="GND"/>
 <wire x1="2.54" y1="83.82" x2="-2.54" y2="83.82" width="0.1524" layer="91"/>
@@
 </segment>
 <segment>
-<pinref part="D1" gate="G$1" pin="VSS"/>
-<pinref part="GND7" gate="1" pin="GND"/>
-<wire x1="134.62" y1="33.02" x2="132.08" y2="33.02" width="0.1524" layer="91"/>
-<wire x1="132.08" y1="33.02" x2="132.08" y2="30.48" width="0.1524" layer="91"/>
-</segment>
-<segment>
-<pinref part="D2" gate="G$1" pin="VSS"/>
-<pinref part="GND8" gate="1" pin="GND"/>
-<wire x1="101.6" y1="33.02" x2="99.06" y2="33.02" width="0.1524" layer="91"/>
-<wire x1="99.06" y1="33.02" x2="99.06" y2="30.48" width="0.1524" layer="91"/>
-</segment>
-<segment>
 <pinref part="C5" gate="G$1" pin="2"/>
 <pinref part="GND9" gate="1" pin="GND"/>
@@
 <pinref part="GND10" gate="1" pin="GND"/>
 <wire x1="127" y1="71.12" x2="127" y2="73.66" width="0.1524" layer="91"/>
+</segment>
+<segment>
+<pinref part="GND4" gate="1" pin="GND"/>
+<wire x1="99.06" y1="33.02" x2="99.06" y2="35.56" width="0.1524" layer="91"/>
+<pinref part="SV1" gate="G$1" pin="1"/>
+<wire x1="99.06" y1="35.56" x2="101.6" y2="35.56" width="0.1524" layer="91"/>
 </segment>
 </net>
@@
 <junction x="45.72" y="91.44"/>
 <wire x1="45.72" y1="91.44" x2="50.8" y2="91.44" width="0.1524" layer="91"/>
-<pinref part="AMS1117" gate="G$1" pin="OUT"/>
-<wire x1="40.64" y1="91.44" x2="43.18" y2="91.44" width="0.1524" layer="91"/>
 <pinref part="P+10" gate="VCC" pin="VCC"/>
 <wire x1="43.18" y1="91.44" x2="45.72" y2="91.44" width="0.1524" layer="91"/>
 <wire x1="50.8" y1="93.98" x2="50.8" y2="91.44" width="0.1524" layer="91"/>
 <junction x="50.8" y="91.44"/>
-<pinref part="AMS1117" gate="G$1" pin="OUT1"/>
+<pinref part="REG" gate="G$1" pin="OUT1"/>
 <wire x1="40.64" y1="93.98" x2="43.18" y2="93.98" width="0.1524" layer="91"/>
 <wire x1="43.18" y1="93.98" x2="43.18" y2="91.44" width="0.1524" layer="91"/>
-<junction x="43.18" y="91.44"/>
 </segment>
 <segment>
@@
 <pinref part="R2" gate="G$1" pin="1"/>
 <wire x1="93.98" y1="40.64" x2="93.98" y2="43.18" width="0.1524" layer="91"/>
-<pinref part="D2" gate="G$1" pin="DOUT"/>
-<wire x1="101.6" y1="40.64" x2="93.98" y2="40.64" width="0.1524" layer="91"/>
+<pinref part="SV1" gate="G$1" pin="3"/>
+<wire x1="93.98" y1="40.64" x2="101.6" y2="40.64" width="0.1524" layer="91"/>
 <junction x="93.98" y="40.64"/>
 </segment>
@@
 <segment>
 <pinref part="C1" gate="G$1" pin="+"/>
-<pinref part="AMS1117" gate="G$1" pin="IN"/>
+<pinref part="REG" gate="G$1" pin="IN"/>
 <wire x1="22.86" y1="91.44" x2="25.4" y2="91.44" width="0.1524" layer="91"/>
 <wire x1="22.86" y1="91.44" x2="22.86" y2="88.9" width="0.1524" layer="91"/>
@@
 <segment>
 <pinref part="P+2" gate="1" pin="+5V"/>
-<wire x1="172.72" y1="45.72" x2="172.72" y2="48.26" width="0.1524" layer="91"/>
-<pinref part="SV1" gate="G$1" pin="3"/>
-<wire x1="175.26" y1="45.72" x2="172.72" y2="45.72" width="0.1524" layer="91"/>
-</segment>
-<segment>
-<pinref part="D1" gate="G$1" pin="VDD"/>
-<pinref part="P+12" gate="1" pin="+5V"/>
-<wire x1="134.62" y1="48.26" x2="132.08" y2="48.26" width="0.1524" layer="91"/>
-<wire x1="132.08" y1="48.26" x2="132.08" y2="50.8" width="0.1524" layer="91"/>
-</segment>
-<segment>
-<pinref part="D2" gate="G$1" pin="VDD"/>
-<pinref part="P+11" gate="1" pin="+5V"/>
-<wire x1="101.6" y1="48.26" x2="99.06" y2="48.26" width="0.1524" layer="91"/>
-<wire x1="99.06" y1="48.26" x2="99.06" y2="50.8" width="0.1524" layer="91"/>
-</segment>
-</net>
-<net name="N$1" class="0">
-<segment>
-<pinref part="D1" gate="G$1" pin="DOUT"/>
-<pinref part="D2" gate="G$1" pin="DIN"/>
-<wire x1="134.62" y1="40.64" x2="132.08" y2="40.64" width="0.1524" layer="91"/>
-</segment>
-</net>
-<net name="N$2" class="0">
-<segment>
-<pinref part="SV1" gate="G$1" pin="1"/>
-<pinref part="D1" gate="G$1" pin="DIN"/>
-<wire x1="175.26" y1="40.64" x2="165.1" y2="40.64" width="0.1524" layer="91"/>
+<wire x1="99.06" y1="43.18" x2="99.06" y2="38.1" width="0.1524" layer="91"/>
+<pinref part="SV1" gate="G$1" pin="2"/>
+<wire x1="99.06" y1="38.1" x2="101.6" y2="38.1" width="0.1524" layer="91"/>
 </segment>
 </net>
@@
 </segment>
 </net>
-<net name="GPIO16" class="0">
-<segment>
-<pinref part="U$1" gate="G$1" pin="GPIO16"/>
-<wire x1="0" y1="43.18" x2="-5.08" y2="43.18" width="0.1524" layer="91"/>
-<label x="-5.08" y="43.18" size="1.27" layer="95" rot="R180" xref="yes"/>
-</segment>
-<segment>
+<net name="GPIO14" class="0">
+<segment>
+<pinref part="U$1" gate="G$1" pin="GPIO14"/>
+<wire x1="0" y1="40.64" x2="-5.08" y2="40.64" width="0.1524" layer="91"/>
+<label x="-5.08" y="40.64" size="1.27" layer="95" rot="R180" xref="yes"/>
+</segment>
+<segment>
